File: Circuit Design/SimpleKnob/SimpleKnob.kicad_sch (KiCad schematic)
At the start: 5 parts, among them J1 Barrel_Jack, M1 Motor_DC, U1 KY-040, U2 L298N

Commit message: Updated README.md
Connections:
- net D2: no longer A1.5 (D2)
Changed lines of the file:
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@@
-    )
-  )
-  (global_label "D2" (shape input) (at 157.48 55.88 180) (fields_autoplaced)
-    (effects (font (size 1.27 1.27)) (justify right))
-    (property "Intersheet References" "${INTERSHEET_REFS}" (id 0) (at 152.5874 55.8006 0)
-      (effects (font (size 1.27 1.27)) (justify right) hide)
     )
   )
